Commit message: Added magnetometer.

File: src/rosbot_description/urdf/rosbot.xacro (robot description, xacro)
@@ -339,3 +339,10 @@
   </joint>
   <link name="range_rr"></link>
+  <joint name="magnetic_joint" type="fixed">
+    <axis xyz="0 1 0" />
+    <origin xyz="0 0 0" rpy="0 0 0" />
+    <parent link="base_link" />
+    <child link="magnetic_link" />
+  </joint>
+  <link name="magnetic_link"></link>
 </robot>

Commit message: Add rangefinders, chg magnetometer noise params.

File: src/rosbot_description/urdf/rosbot.xacro (robot description, xacro)
@@ -339,4 +339,18 @@
   </joint>
   <link name="range_rr"></link>
+  <joint name="range_ri_joint" type="fixed">
+    <axis xyz="0 1 0" />
+    <origin xyz="0.0 -0.075 0.0515" rpy="0 0 -1.57 "/>
+    <parent link="base_link"/>
+    <child link="range_ri"/>
+  </joint>
+  <link name="range_ri"></link>
+  <joint name="range_le_joint" type="fixed">
+    <axis xyz="0 1 0" />
+    <origin xyz="0.0 0.075 0.0515" rpy="0 0 1.57 "/>
+    <parent link="base_link"/>
+    <child link="range_le"/>
+  </joint>
+  <link name="range_le"></link>
   <joint name="magnetic_joint" type="fixed">
     <axis xyz="0 1 0" />
